File: Hardware/EKG/EKG.sch (KiCad schematic (older format))
At the start: 11 parts, among them U2 MAX30003

Commit message: Recent route 5/29
Parts:
- C10, C12, C14, C6, C7, C8: footprint (none) -> Capacitors_SMD:C_0402
- C11, C13, C9: footprint (none) -> Capacitors_SMD:C_0603_HandSoldering
- R13: renamed from R15; footprint (none) -> Resistors_SMD:R_0603_HandSoldering
- U2: footprint (none) -> Housings_DFN_QFN:QFN-28-1EP_5x5mm_Pitch0.5mm
Changed lines of the file:
@@
 $Descr A4 11693 8268
 encoding utf-8
-Sheet 3 4
+Sheet 4 4
 Title ""
 Date ""
@@
 F 0 "U4" H 6800 2900 60  0000 C CNN
 F 1 "MAX30003" H 6800 3000 60  0000 C CNN
-F 2 "" H 5800 3850 60  0001 C CNN
+F 2 "Housings_DFN_QFN:QFN-28-1EP_5x5mm_Pitch0.5mm" H 5800 3850 60  0001 C CNN
 F 3 "" H 5800 3850 60  0001 C CNN
 	1    5800 3850
@@
 F 0 "C29" H 3960 3770 50  0000 L CNN
 F 1 "10uF" H 3960 3620 50  0000 L CNN
-F 2 "" H 3950 3700 50  0001 C CNN
+F 2 "Capacitors_SMD:C_0603_HandSoldering" H 3950 3700 50  0001 C CNN
 F 3 "" H 3950 3700 50  0001 C CNN
 	1    3950 3700
@@
 F 0 "C30" H 4360 3870 50  0000 L CNN
 F 1 "1uF" H 4360 3720 50  0000 L CNN
-F 2 "" H 4350 3800 50  0001 C CNN
+F 2 "Capacitors_SMD:C_0402" H 4350 3800 50  0001 C CNN
 F 3 "" H 4350 3800 50  0001 C CNN
 	1    4350 3800
@@
 F 0 "C31" H 4710 3970 50  0000 L CNN
 F 1 "10uF" H 4710 3820 50  0000 L CNN
-F 2 "" H 4700 3900 50  0001 C CNN
+F 2 "Capacitors_SMD:C_0603_HandSoldering" H 4700 3900 50  0001 C CNN
 F 3 "" H 4700 3900 50  0001 C CNN
 	1    4700 3900
@@
 F 0 "C32" H 7460 4370 50  0000 L CNN
 F 1 "1000pF" H 7460 4220 50  0000 L CNN
-F 2 "" H 7450 4300 50  0001 C CNN
+F 2 "Capacitors_SMD:C_0402" H 7450 4300 50  0001 C CNN
 F 3 "" H 7450 4300 50  0001 C CNN
 	1    7450 4300
@@
 $EndComp
 $Comp
-L Earth #PWR026
+L Earth #PWR23
 U 1 1 5AE78D48
 P 7450 4500
-AR Path="/5AE78932/5AE78D48" Ref="#PWR026"  Part="1"
-AR Path="/5AEA43E2/5AE78D48" Ref="#PWR036"  Part="1"
-AR Path="/5AEA8503/5AE78D48" Ref="#PWR046"  Part="1"
-F 0 "#PWR046" H 7450 4250 50  0001 C CNN
+AR Path="/5AE78932/5AE78D48" Ref="#PWR23"  Part="1"
+AR Path="/5AEA43E2/5AE78D48" Ref="#PWR33"  Part="1"
+AR Path="/5AEA8503/5AE78D48" Ref="#PWR43"  Part="1"
+F 0 "#PWR43" H 7450 4250 50  0001 C CNN
 F 1 "Earth" H 7450 4350 50  0001 C CNN
 F 2 "" H 7450 4500 50  0001 C CNN
@@
 F 0 "C25" H 5160 2470 50  0000 L CNN
 F 1 "1uF" H 5160 2320 50  0000 L CNN
-F 2 "" H 5150 2400 50  0001 C CNN
+F 2 "Capacitors_SMD:C_0402" H 5150 2400 50  0001 C CNN
 F 3 "" H 5150 2400 50  0001 C CNN
 	1    5150 2400
@@
 F 0 "C27" H 6510 2470 50  0000 L CNN
 F 1 "10uF" H 6510 2320 50  0000 L CNN
-F 2 "" H 6500 2400 50  0001 C CNN
+F 2 "Capacitors_SMD:C_0603_HandSoldering" H 6500 2400 50  0001 C CNN
 F 3 "" H 6500 2400 50  0001 C CNN
 	1    6500 2400
@@
 F 0 "C24" H 4810 2470 50  0000 L CNN
 F 1 "1uF" H 4810 2320 50  0000 L CNN
-F 2 "" H 4800 2400 50  0001 C CNN
+F 2 "Capacitors_SMD:C_0402" H 4800 2400 50  0001 C CNN
 F 3 "" H 4800 2400 50  0001 C CNN
 	1    4800 2400
@@
 $EndComp
 $Comp
-L Earth #PWR027
+L Earth #PWR19
 U 1 1 5AE78D6A
 P 5150 2600
-AR Path="/5AE78932/5AE78D6A" Ref="#PWR027"  Part="1"
-AR Path="/5AEA43E2/5AE78D6A" Ref="#PWR037"  Part="1"
-AR Path="/5AEA8503/5AE78D6A" Ref="#PWR047"  Part="1"
-F 0 "#PWR047" H 5150 2350 50  0001 C CNN
+AR Path="/5AE78932/5AE78D6A" Ref="#PWR19"  Part="1"
+AR Path="/5AEA43E2/5AE78D6A" Ref="#PWR29"  Part="1"
+AR Path="/5AEA8503/5AE78D6A" Ref="#PWR39"  Part="1"
+F 0 "#PWR39" H 5150 2350 50  0001 C CNN
 F 1 "Earth" H 5150 2450 50  0001 C CNN
 F 2 "" H 5150 2600 50  0001 C CNN
@@
 $EndComp
 $Comp
-L Earth #PWR028
+L Earth #PWR18
 U 1 1 5AE78D70
 P 4800 2600
-AR Path="/5AE78932/5AE78D70" Ref="#PWR028"  Part="1"
-AR Path="/5AEA43E2/5AE78D70" Ref="#PWR038"  Part="1"
-AR Path="/5AEA8503/5AE78D70" Ref="#PWR048"  Part="1"
-F 0 "#PWR048" H 4800 2350 50  0001 C CNN
+AR Path="/5AE78932/5AE78D70" Ref="#PWR18"  Part="1"
+AR Path="/5AEA43E2/5AE78D70" Ref="#PWR28"  Part="1"
+AR Path="/5AEA8503/5AE78D70" Ref="#PWR38"  Part="1"
+F 0 "#PWR38" H 4800 2350 50  0001 C CNN
 F 1 "Earth" H 4800 2450 50  0001 C CNN
 F 2 "" H 4800 2600 50  0001 C CNN
@@
 $EndComp
 $Comp
-L Earth #PWR029
+L Earth #PWR21
 U 1 1 5AE78D76
 P 6500 2600
-AR Path="/5AE78932/5AE78D76" Ref="#PWR029"  Part="1"
-AR Path="/5AEA43E2/5AE78D76" Ref="#PWR039"  Part="1"
-AR Path="/5AEA8503/5AE78D76" Ref="#PWR049"  Part="1"
-F 0 "#PWR049" H 6500 2350 50  0001 C CNN
+AR Path="/5AE78932/5AE78D76" Ref="#PWR21"  Part="1"
+AR Path="/5AEA43E2/5AE78D76" Ref="#PWR31"  Part="1"
+AR Path="/5AEA8503/5AE78D76" Ref="#PWR41"  Part="1"
+F 0 "#PWR41" H 6500 2350 50  0001 C CNN
 F 1 "Earth" H 6500 2450 50  0001 C CNN
 F 2 "" H 6500 2600 50  0001 C CNN
@@
 $EndComp
 $Comp
-L +1V8 #PWR030
+L +1V8 #PWR15
 U 1 1 5AE78D7C
 P 4800 2050
-AR Path="/5AE78932/5AE78D7C" Ref="#PWR030"  Part="1"
-AR Path="/5AEA43E2/5AE78D7C" Ref="#PWR040"  Part="1"
-AR Path="/5AEA8503/5AE78D7C" Ref="#PWR050"  Part="1"
-F 0 "#PWR050" H 4800 1900 50  0001 C CNN
+AR Path="/5AE78932/5AE78D7C" Ref="#PWR15"  Part="1"
+AR Path="/5AEA43E2/5AE78D7C" Ref="#PWR25"  Part="1"
+AR Path="/5AEA8503/5AE78D7C" Ref="#PWR35"  Part="1"
+F 0 "#PWR35" H 4800 1900 50  0001 C CNN
 F 1 "+1V8" H 4800 2190 50  0000 C CNN
 F 2 "" H 4800 2050 50  0001 C CNN
@@
 F 0 "C28" H 4450 3250 50  0000 L CNN
 F 1 "1uF" H 4400 3150 50  0000 L CNN
-F 2 "" H 4650 3200 50  0001 C CNN
+F 2 "Capacitors_SMD:C_0402" H 4650 3200 50  0001 C CNN
 F 3 "" H 4650 3200 50  0001 C CNN
 	1    4650 3200
@@
 $EndComp
 $Comp
-L R_Small R15
+L R_Small R13
 U 1 1 5AE78D92
 P 3550 3550
-AR Path="/5AE78932/5AE78D92" Ref="R15"  Part="1"
-AR Path="/5AEA43E2/5AE78D92" Ref="R16"  Part="1"
-AR Path="/5AEA8503/5AE78D92" Ref="R17"  Part="1"
-F 0 "R17" V 3650 3500 50  0000 L CNN
+AR Path="/5AE78932/5AE78D92" Ref="R13"  Part="1"
+AR Path="/5AEA43E2/5AE78D92" Ref="R14"  Part="1"
+AR Path="/5AEA8503/5AE78D92" Ref="R15"  Part="1"
+F 0 "R15" V 3650 3500 50  0000 L CNN
 F 1 "499k" V 3450 3450 50  0000 L CNN
-F 2 "" H 3550 3550 50  0001 C CNN
+F 2 "Resistors_SMD:R_0603_HandSoldering" H 3550 3550 50  0001 C CNN
 F 3 "" H 3550 3550 50  0001 C CNN
 	1    3550 3550
@@
 F 0 "C26" H 5410 2470 50  0000 L CNN
 F 1 "0.1uF" H 5410 2320 50  0000 L CNN
-F 2 "" H 5400 2400 50  0001 C CNN
+F 2 "Capacitors_SMD:C_0402" H 5400 2400 50  0001 C CNN
 F 3 "" H 5400 2400 50  0001 C CNN
 	1    5400 2400
@@
 $EndComp
 $Comp
-L Earth #PWR031
+L Earth #PWR20
 U 1 1 5AE78DA8
 P 5400 2600
-AR Path="/5AE78932/5AE78DA8" Ref="#PWR031"  Part="1"
-AR Path="/5AEA43E2/5AE78DA8" Ref="#PWR041"  Part="1"
-AR Path="/5AEA8503/5AE78DA8" Ref="#PWR051"  Part="1"
-F 0 "#PWR051" H 5400 2350 50  0001 C CNN
+AR Path="/5AE78932/5AE78DA8" Ref="#PWR20"  Part="1"
+AR Path="/5AEA43E2/5AE78DA8" Ref="#PWR30"  Part="1"
+AR Path="/5AEA8503/5AE78DA8" Ref="#PWR40"  Part="1"
+F 0 "#PWR40" H 5400 2350 50  0001 C CNN
 F 1 "Earth" H 5400 2450 50  0001 C CNN
 F 2 "" H 5400 2600 50  0001 C CNN
@@
 AVDD
 $Comp
-L +1V8 #PWR032
+L +1V8 #PWR16
 U 1 1 5AE78DB7
 P 4800 2050
-AR Path="/5AE78932/5AE78DB7" Ref="#PWR032"  Part="1"
-AR Path="/5AEA43E2/5AE78DB7" Ref="#PWR042"  Part="1"
-AR Path="/5AEA8503/5AE78DB7" Ref="#PWR052"  Part="1"
-F 0 "#PWR052" H 4800 1900 50  0001 C CNN
+AR Path="/5AE78932/5AE78DB7" Ref="#PWR16"  Part="1"
+AR Path="/5AEA43E2/5AE78DB7" Ref="#PWR26"  Part="1"
+AR Path="/5AEA8503/5AE78DB7" Ref="#PWR36"  Part="1"
+F 0 "#PWR36" H 4800 1900 50  0001 C CNN
 F 1 "+1V8" H 4800 2190 50  0000 C CNN
 F 2 "" H 4800 2050 50  0001 C CNN
@@
 $EndComp
 $Comp
-L Earth #PWR033
+L Earth #PWR24
 U 1 1 5AE78DBD
 P 5800 5200
-AR Path="/5AE78932/5AE78DBD" Ref="#PWR033"  Part="1"
-AR Path="/5AEA43E2/5AE78DBD" Ref="#PWR043"  Part="1"
-AR Path="/5AEA8503/5AE78DBD" Ref="#PWR053"  Part="1"
-F 0 "#PWR053" H 5800 4950 50  0001 C CNN
+AR Path="/5AE78932/5AE78DBD" Ref="#PWR24"  Part="1"
+AR Path="/5AEA43E2/5AE78DBD" Ref="#PWR34"  Part="1"
+AR Path="/5AEA8503/5AE78DBD" Ref="#PWR44"  Part="1"
+F 0 "#PWR44" H 5800 4950 50  0001 C CNN
 F 1 "Earth" H 5800 5050 50  0001 C CNN
 F 2 "" H 5800 5200 50  0001 C CNN
@@
 $EndComp
 $Comp
-L +3V3 #PWR034
+L +3V3 #PWR17
 U 1 1 5AE79031
 P 6500 2050
-AR Path="/5AE78932/5AE79031" Ref="#PWR034"  Part="1"
-AR Path="/5AEA43E2/5AE79031" Ref="#PWR044"  Part="1"
-AR Path="/5AEA8503/5AE79031" Ref="#PWR054"  Part="1"
-F 0 "#PWR054" H 6500 1900 50  0001 C CNN
+AR Path="/5AE78932/5AE79031" Ref="#PWR17"  Part="1"
+AR Path="/5AEA43E2/5AE79031" Ref="#PWR27"  Part="1"
+AR Path="/5AEA8503/5AE79031" Ref="#PWR37"  Part="1"
+F 0 "#PWR37" H 6500 1900 50  0001 C CNN
 F 1 "+3V3" H 6500 2190 50  0000 C CNN
 F 2 "" H 6500 2050 50  0001 C CNN
@@
 $EndComp
 $Comp
-L Earth #PWR035
+L Earth #PWR22
 U 1 1 5AE7BA34
 P 4350 4150
-AR Path="/5AE78932/5AE7BA34" Ref="#PWR035"  Part="1"
-AR Path="/5AEA43E2/5AE7BA34" Ref="#PWR045"  Part="1"
-AR Path="/5AEA8503/5AE7BA34" Ref="#PWR055"  Part="1"
-F 0 "#PWR055" H 4350 3900 50  0001 C CNN
+AR Path="/5AE78932/5AE7BA34" Ref="#PWR22"  Part="1"
+AR Path="/5AEA43E2/5AE7BA34" Ref="#PWR32"  Part="1"
+AR Path="/5AEA8503/5AE7BA34" Ref="#PWR42"  Part="1"
+F 0 "#PWR42" H 4350 3900 50  0001 C CNN
 F 1 "Earth" H 4350 4000 50  0001 C CNN
 F 2 "" H 4350 4150 50  0001 C CNN
