File: Hardware/EKG/EKGProject.sch (KiCad schematic (older format))
At the start: 29 parts, among them J1 Screw_Terminal_01x01, J2 Screw_Terminal_01x01, J3 Screw_Terminal_01x01, J4 Screw_Terminal_01x01, J5 Conn_01x12, J6 Conn_01x16, J7 Conn_01x10, U1 MAX1726EUK18+

Commit message: Add files via upload
Updated schematic
Final version V1
Parts:
- added J1: Screw_Terminal_01x01, symbol Screw_Terminal_01x01
- added J11: Conn_01x04, symbol Conn_01x04
- added J12: Conn_02x02_Counter_Clockwise, symbol Conn_02x02_Counter_Clockwise
- added J13: Conn_01x02, symbol Conn_01x02
- added J4, J7: Conn_01x01, symbol Conn_01x01
- R13, R14: value 0 -> 1k
- renumbered J7 to J10, J1 to J2, J2 to J3, J3 to J5, J4 to J6, J5 to J8, J6 to J9
Connections:
- net +1V8: now also J11.4 (Pin_4)
- net +3V3: now also J11.3 (Pin_3)
- net ECGP_2_R: now also J4.1 (Pin_1)
- net ECGP_3_R: now also J7.1 (Pin_1)
- net Earth: now also J12.3 (Pin_3)
- net FCLK: now also J9.15 (Pin_15)
- net VBAT: now also J11.1 (Pin_1), J12.4 (Pin_4)
- net PP3V3_EN: now reaches J8.2 (Pin_2)
- net PP3V3_EN: now also J10.8 (Pin_8)
- net VUSB: now reaches J8.3 (Pin_3)
- net VUSB: now also J11.2 (Pin_2)
- removed net GPIO_1: J10.8 (Pin_8), J9.15 (Pin_15)
- new net GND_CONN: J12.2 (Pin_2), J13.1 (Pin_1)
- new net VBAT_CONN: J12.1 (Pin_1), J13.2 (Pin_2)
- new net VCM_1: J1.1 (Pin_1)
- no-connect marks 5 -> 1

Commit message: Recent route 5/29
Parts:
- removed D1, D2: LED, symbol LED
- removed J10: Conn_01x10, symbol Conn_01x10
- removed J12: Conn_02x02_Counter_Clockwise, symbol Conn_02x02_Counter_Clockwise
- removed J13: Conn_01x02, symbol Conn_01x02
- removed R13, R14: 1k, symbol R_Small
- added R16: 10k, Resistors_SMD:R_0805_HandSoldering, symbol R_Small
- C1, C3, C4, C5, R1, R10, R11, R12, R2, R3, R4, R5, R6, R7, R8, R9: footprint (none) -> Resistors_SMD:R_0805_HandSoldering
- C2: footprint (none) -> Capacitors_SMD:C_0402
- J1, J2, J3, J4, J5, J6, J7: footprint (none) -> Wire_Pads:SolderWirePad_single_1-5mmDrill
- J10: renamed from J11; footprint (none) -> Pin_Headers:Pin_Header_Straight_1x04_Pitch2.54mm
- J8: footprint (none) -> Pin_Headers:Pin_Header_Straight_1x12_Pitch2.54mm
- J9: footprint (none) -> Pin_Headers:Pin_Header_Straight_1x16_Pitch2.54mm
- U1: footprint (none) -> TO_SOT_Packages_SMD:TSOT-23-5_HandSoldering
Connections:
- net +1V8: no longer J10.4 (Pin_4)
- net +3V3: now also R16.1; no longer J10.3 (Pin_3)
- net ECGP_2_R: no longer J4.1 (Pin_1)
- net ECGP_3_R: no longer J7.1 (Pin_1)
- net Earth: now also J10.1 (Pin_1), J10.2 (Pin_2), J10.3 (Pin_3), J10.4 (Pin_4); no longer J9.16 (Pin_16)
- net GPIO_14: now also R16.2
- net VBAT: no longer names the net of J8.1 (Pin_1)
- net VBAT: no longer J10.1 (Pin_1)
- net VUSB: no longer names the net of J8.3 (Pin_3)
- net VUSB: no longer J10.2 (Pin_2)
- new net VCM_2: J4.1 (Pin_1)
- new net VCM_3: J7.1 (Pin_1)
- no-connect marks 1 -> 11
Other:
- moved on the sheet: J10
