File: Hardware/EKG/EKGProject.kicad_pcb (KiCad board)
At the start: 2 copper layers, 62 parts, among them J1 Screw_Terminal_01x01, J10 Conn_01x04, J2 Screw_Terminal_01x01, J3 Screw_Terminal_01x01, J4 Conn_01x01, J5 Screw_Terminal_01x01, J6 Screw_Terminal_01x01, J7 Conn_01x01, J8 Conn_01x12, J9 Conn_01x16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

Commit message: updated super close finished layout
Parts:
- moved R16 137.0 mm to (125.3, 88.6), turned to 0 degrees
- moved R4 129.7 mm to (136.8, 95.9)
- moved R11 110.6 mm to (165.7, 77.0)
- moved R9 97.7 mm to (165.6, 69.3)
- moved R12 91.8 mm to (170.7, 69.3)
- moved R5 88.5 mm to (124.2, 99.8), turned to 270 degrees
- moved R3 83.9 mm to (175.8, 69.3)
- moved R2 79.5 mm to (124.2, 93.5), turned to 270 degrees
- moved C2 78.8 mm to (121.2, 108.6)
- moved U1 78.0 mm to (127.1, 106.7)
- moved R8 74.7 mm to (180.8, 69.3)
- moved J1 32.0 mm to (137.2, 132.0)
- moved J4 31.9 mm to (158.9, 132.0)
- moved J7 25.7 mm to (203.1, 129.4)
- moved R15 22.8 mm to (178.6, 122.3)
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Routing:
- net /MISO: track 0.00 -> 101.6 mm, vias 0 -> 3
- net +3V3: track 8.77 -> 106.2 mm, vias 0 -> 5
- net +1V8: track 30.0 -> 112.2 mm, vias 0 -> 9
- net /CS_3: track 0.00 -> 76.3 mm, vias 0 -> 1
- net /FCLK: track 32.6 -> 99.5 mm, vias 2 -> 4
- net /INT2B_1_R: track 0.00 -> 62.9 mm, vias 0 -> 2
- net /SCLK: track 31.6 -> 88.5 mm, vias 2 -> 7
- net /CS_2: track 0.00 -> 56.7 mm, vias 0 -> 2
- net /INTB_2_R: track 0.00 -> 51.2 mm
- net /CS_1: track 0.00 -> 50.2 mm
- net /INT2B_2_R: track 0.00 -> 49.5 mm
- net /INTB_1: track 0.00 -> 45.1 mm
- net /INTB_3_R: track 0.00 -> 44.7 mm, vias 0 -> 2
- net /INT2B_3_R: track 0.00 -> 40.5 mm, vias 0 -> 4
- net /MOSI: track 62.2 -> 98.1 mm, vias 0 -> 5
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Other:
- net class Default: clearance 0.2 -> 0.19
- net class power added: clearance 0.19, trace_width 0.5, via_dia 0.6, via_drill 0.4
- rule trace_clearance: 0.2 -> 0.19
- rule trace_min: 0.2 -> 0.0889
- rule via_min_size: 0.4 -> 0.2

Commit message: hopefully final board layout?
Parts:
- added REF**: MountingHole_4mm_Pad, Mounting_Holes:MountingHole_4mm_Pad, F.Cu at (201.1, 130.6)
- added REF**: MountingHole_4mm_Pad, Mounting_Holes:MountingHole_4mm_Pad, F.Cu at (119.8, 130.6)
- added REF**: MountingHole_4mm_Pad, Mounting_Holes:MountingHole_4mm_Pad, F.Cu at (201.1, 62.4)
- added REF**: MountingHole_4mm_Pad, Mounting_Holes:MountingHole_4mm_Pad, F.Cu at (119.8, 62.4)
- moved J5 15.8 mm to (202.2, 104.5)
- moved J7 13.2 mm to (202.2, 116.3)
- moved J10 8.42 mm to (190.7, 76.2)
- moved J6 4.85 mm to (118.7, 115.5)
- moved R7 2.20 mm to (191.9, 119.9)
- moved J1 0.07 mm to (137.2, 131.9)
- moved J2 0.07 mm to (148.3, 131.9)
- moved J3 0.07 mm to (169.8, 131.9)
- moved J4 0.07 mm to (158.9, 131.9)
Routing:
- net /ECGP_3: track 7.79 -> 19.0 mm
- net +1V8: track 112.2 -> 116.7 mm, vias 9 -> 11
- net /ECGP_3_R: track 11.6 -> 9.33 mm
- net /ECGN: track 6.45 -> 8.26 mm
- net /VCM_3: track 27.1 -> 28.0 mm
- net /INTB_1: track 45.1 -> 46.0 mm
- net Earth: track 34.2 -> 33.4 mm, vias 10 -> 133
- net /SHDN_L_R: track 15.0 -> 15.6 mm
Other:
- board outline added: 93.5 x 80.8 mm

Commit message: DFM quick check
Routing:
- net +3V3: track 106.2 -> 45.2 mm, vias 5 -> 4
- net /MISO: track 101.6 -> 67.3 mm, vias 3 -> 2
- net /MOSI: track 98.1 -> 75.1 mm, vias 5 -> 4
- net +1V8: track 116.7 -> 107.5 mm
- net Earth: track 33.4 -> 32.3 mm, vias 133 -> 15
- net /FCLK: track 99.5 -> 98.7 mm
- net /INTB_2_R: track 51.2 -> 50.7 mm
Other:
- board size 93.5 x 80.8 mm -> 94 x 81.5 mm
