File: Hardware/EKG/EKGProject.kicad_pcb (KiCad board)
At the start: 2 copper layers, 94 x 81.5 mm, 66 parts, among them J1 Screw_Terminal_01x01, J10 Conn_01x04, J2 Screw_Terminal_01x01, J3 Screw_Terminal_01x01, J4 Conn_01x01, J5 Screw_Terminal_01x01, J6 Screw_Terminal_01x01, J7 Conn_01x01, J8 Conn_01x12, J9 Conn_01x16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

Commit message: one more time DFM lets goooo
Routing:
- net /SCLK: vias 7 -> 6
Changed lines of the file:
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@@
   (segment (start 143.480269 114.469161) (end 143.480269 118.016769) (width 0.25) (layer F.Cu) (net 1) (status 30))
   (segment (start 143.480269 118.016769) (end 143.51 118.0465) (width 0.25) (layer F.Cu) (net 1) (status 30))
+  (segment (start 144.930269 113.519161) (end 144.930269 113.688269) (width 0.25) (layer F.Cu) (net 2))
   (segment (start 166.457625 113.519161) (end 166.457625 113.755175) (width 0.25) (layer F.Cu) (net 2))
   (segment (start 125.417 106.68) (end 124.167 106.68) (width 0.25) (layer F.Cu) (net 2))
@@
   (segment (start 145.923 90.297) (end 145.923 101.219) (width 0.25) (layer F.Cu) (net 50))
   (segment (start 146.304 89.916) (end 145.923 90.297) (width 0.25) (layer F.Cu) (net 50))
-  (via (at 145.923 101.219) (size 0.6) (drill 0.4) (layers F.Cu B.Cu) (net 50))
   (segment (start 146.431 86.614) (end 146.431 89.789) (width 0.25) (layer B.Cu) (net 50))
   (segment (start 146.431 89.789) (end 146.304 89.916) (width 0.25) (layer B.Cu) (net 50))
